File: PWMGenerator_EuniceF/PWMGenerator_EuniceF.kicad_sch (KiCad schematic)
At the start: 12 parts, among them J1 Conn_01x03_Pin, Q1 NPN, Q2 NPN, Q3 PNP, Q4 PNP, SW1 SW_SPST, U1 LM7805_TO220, U2 LM339

Commit message: PWMGenerator
Parts:
- removed R2: Potentiometer, symbol Simulation_SPICE:Potentiometer
- removed V1: VSIN, symbol Simulation_SPICE:VSIN
- added C1: 220u, Capacitor_THT:CP_Radial_D10.0mm_P5.00mm_P7.50mm, symbol Device:C_Polarized_Small_US
- added C2: 10u, Capacitor_THT:CP_Radial_D10.0mm_P5.00mm_P7.50mm, symbol Device:C_Polarized_Small_US
- added C3: 0.1u, Capacitor_SMD:C_0805_2012Metric, symbol Device:C
- added D2, D4, D5, D6: 1N4005G, Diode_SMD:D_0805_2012Metric, symbol Diode:1N4005
- added D3: 1N4005G, Diode_THT:D_DO-41_SOD81_P10.16mm_Horizontal, symbol Diode:1N4005
- added J2: Barrel_Jack, Connector_BarrelJack:BarrelJack_CUI_PJ-063AH_Horizontal, symbol Connector:Barrel_Jack
- added R10: 8.2k, Resistor_SMD:R_0805_2012Metric, symbol Device:R_US
- added R11: 180, Resistor_SMD:R_0805_2012Metric, symbol Device:R_US
- added R2: 1M, Resistor_SMD:R_0805_2012Metric, symbol Device:R_US
- added R3: 330, Resistor_SMD:R_0805_2012Metric, symbol Device:R_US
- added R4: 10k, Resistor_SMD:R_0805_2012Metric, symbol Device:R_US
- added R5: 220k, Resistor_SMD:R_0805_2012Metric, symbol Device:R_US
- added R6: 390, Resistor_SMD:R_0805_2012Metric, symbol Device:R_US
- added R7: 22k, Resistor_SMD:R_0805_2012Metric, symbol Device:R_US
- added R8: 2.2k, Resistor_SMD:R_0805_2012Metric, symbol Device:R_US
- added RV1: 5k, Potentiometer_THT:Potentiometer_ACP_CA14-H2,5_Horizontal, symbol Device:R_Potentiometer_US
- D1: value LED -> LED_GREEN; footprint (none) -> LED_THT:LED_D5.0mm_GREEN
- J1: footprint (none) -> Connector_PinHeader_2.54mm:PinHeader_1x03_P2.54mm_Horizontal
- Q1, Q2: value NPN -> 2N3904; footprint (none) -> Package_TO_SOT_SMD:SOT-23
- Q3, Q4: value PNP -> 2N3906; footprint (none) -> Package_TO_SOT_SMD:SOT-23
- R1: value R_US -> 2.2k; footprint (none) -> Resistor_SMD:R_0805_2012Metric
- SW1: footprint (none) -> Button_Switch_SMD:SW_DIP_SPSTx01_Slide_6.7x4.1mm_W6.73mm_P2.54mm_LowProfile_JPin
- U1: footprint Package_TO_SOT_THT:TO-220-3_Vertical -> Package_TO_SOT_THT:TO-220-3_Horizontal_TabDown
- U2: footprint (none) -> Package_SO:SOIC-14_3.9x8.7mm_P1.27mm
Connections:
- net GND is gone; now on net GNDPWR: D1.1 (K)
- net GNDPWR: now also J1.3 (Pin_3), Q1.3 (E), Q2.3 (E), R1.2, C3.2, D2.2 (A), D4.2 (A), J2.2, R11.2, R6.2, RV1.2, RV1.3; no longer U1.2 (GND)
- net VCC 5V: now also J1.2 (Pin_2), Q4.3 (E), C2.1, R3.1, R4.1, R5.1, R7.1, R8.1; no longer R1.1
- net at SW1.1 (A): now also D4.1 (K), D6.2 (A), J2.1
- net at SW1.2 (B): now also D2.1 (K), D3.2 (A)
- net at U2.2: now also R10.1
- net at U2.4 (-): now also Q1.1 (C), Q3.1 (C), C3.1
- net at U2.5 (+): now also R8.2, RV1.1
- net at D1.2 (A): now also R3.2; no longer R1.2
- net at Q1.2 (B): now also Q2.1 (C), R4.2
- net at Q3.2 (B): now also R5.2, R6.1
- net at Q3.3 (E): now also R7.2
- net at U1.1 (VI): now also C1.1, D5.1 (K)
- net PWM: now reaches Q4.1 (C)
- net PWM: now also J1.1 (Pin_1), R11.1
- net at Q4.2 (B): now also R10.2
- net at Q2.2 (B): now also R2.2
- new net: D3.1 (K), D5.2 (A), D6.1 (K), R1.1, R2.1
- new net: C1.2, C2.2, U1.2 (GND)
Other:
- moved on the sheet: D1, J1, Q1, Q2, Q3, Q4, SW1, U1, U2A

Commit message: PCB Part B
Parts:
- removed Q1, Q2: 2N3904, Package_TO_SOT_SMD:SOT-23, symbol Simulation_SPICE:NPN
- removed Q3, Q4: 2N3906, Package_TO_SOT_SMD:SOT-23, symbol Simulation_SPICE:PNP
- added F1: Polyfuse, symbol Device:Polyfuse
- added Q1, Q2: 2N3906, Package_TO_SOT_SMD:SOT-23, symbol Transistor_BJT:2N3906
- added Q5, Q6: 2N3904, Package_TO_SOT_SMD:SOT-23, symbol Device:Q_NPN
Connections:
- net PWM: now also Q2.3 (C)
- net VCC 5V: now also Q2.1 (E)
- net at D2.1 (K), D3.2 (A): now also F1.2; no longer SW1.2 (B)
- net at C3.1, U2.4 (-): now also Q1.3 (C), Q6.C
- net at R4.2: now also Q5.C, Q6.B
- net at R2.2: now also Q5.B
- net at R5.2, R6.1: now also Q1.2 (B)
- net at R7.2: now also Q1.1 (E)
- net at R10.2: now also Q2.2 (B)
- net GNDPWR renamed GND
- net GND: now also Q5.E, Q6.E
- new net: F1.1, SW1.2 (B)
- new net +12V: U2.3 (V+)
- new net -12V: U2.12 (V-)
- no-connect marks 0 -> 9
Other:
- moved on the sheet: D1, SW1

Commit message: PCB Part B
Parts:
- added unit 2 of U2
- added unit 3 of U2
- added unit 4 of U2
- added unit 5 of U2
- D1: footprint LED_THT:LED_D5.0mm_GREEN -> LED_THT:LED_D5.0mm-4_RGB
- F1: value Polyfuse -> NANOSMDC016F-2; footprint (none) -> lib:RESC3115X65N
Connections:
- net +12V: now also U2.3 (V+); no longer U2.3 (V+)
- net -12V: now also U2.12 (V-); no longer U2.12 (V-)
Changed lines of the file:
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@@
 	(wire
 		(pts
+			(xy 111.76 88.9) (xy 110.49 88.9)
+		)
+		(stroke
+			(width 0)
+			(type default)
+		)
+	)
+	(wire
+		(pts
 			(xy 224.79 162.56) (xy 215.9 162.56)
 		)
@@
 	(wire
 		(pts
+			(xy 123.19 81.28) (xy 128.27 81.28)
+		)
+		(stroke
+			(width 0)
+			(type default)
+		)
+	)
+	(wire
+		(pts
 			(xy 185.42 175.26) (xy 190.5 175.26)
 		)
@@
 	(wire
 		(pts
+			(xy 128.27 81.28) (xy 128.27 99.06)
+		)
+		(stroke
+			(width 0)
+			(type default)
+		)
+	)
+	(wire
+		(pts
 			(xy 208.28 177.8) (xy 205.74 177.8)
 		)
@@
 	(wire
 		(pts
-			(xy 116.84 88.9) (xy 110.49 88.9)
-		)
-		(stroke
-			(width 0)
-			(type default)
-		)
-	)
-	(wire
-		(pts
 			(xy 119.38 128.27) (xy 119.38 133.35)
 		)
@@
 	(wire
 		(pts
-			(xy 184.15 101.6) (xy 173.99 101.6)
+			(xy 111.76 81.28) (xy 111.76 88.9)
 		)
 		(stroke
@@
 	(wire
 		(pts
-			(xy 128.27 88.9) (xy 124.46 88.9)
+			(xy 184.15 101.6) (xy 173.99 101.6)
 		)
 		(stroke
@@
 	(wire
 		(pts
-			(xy 128.27 88.9) (xy 128.27 99.06)
+			(xy 250.19 69.85) (xy 245.11 69.85)
 		)
 		(stroke
@@
 	(wire
 		(pts
-			(xy 250.19 69.85) (xy 245.11 69.85)
+			(xy 128.27 99.06) (xy 135.89 99.06)
 		)
 		(stroke
@@
 	(wire
 		(pts
-			(xy 128.27 99.06) (xy 135.89 99.06)
+			(xy 215.9 125.73) (xy 215.9 133.35)
 		)
 		(stroke
@@
 	(wire
 		(pts
-			(xy 215.9 125.73) (xy 215.9 133.35)
+			(xy 111.76 81.28) (xy 115.57 81.28)
 		)
 		(stroke
@@
 			)
 		)
-		(property "Footprint" "LED_THT:LED_D5.0mm_GREEN"
+		(property "Footprint" "LED_THT:LED_D5.0mm-4_RGB"
 			(at 184.15 119.38 0)
 			(hide yes)
@@
 	)
 	(symbol
-		(lib_id "Device:Polyfuse")
-		(at 120.65 88.9 90)
-		(unit 1)
-		(body_style 1)
-		(exclude_from_sim no)
-		(in_bom yes)
-		(on_board yes)
-		(in_pos_files yes)
-		(dnp no)
-		(fields_autoplaced yes)
-		(property "Reference" "F1"
-			(at 120.65 82.55 90)
-			(show_name no)
-			(do_not_autoplace no)
-			(effects
-				(font
-					(size 1.27 1.27)
-				)
-			)
-		)
-		(property "Value" "Polyfuse"
-			(at 120.65 85.09 90)
-			(show_name no)
-			(do_not_autoplace no)
-			(effects
-				(font
-					(size 1.27 1.27)
-				)
-			)
-		)
-		(property "Footprint" ""
-			(at 125.73 87.63 0)
-			(hide yes)
-			(show_name no)
-			(do_not_autoplace no)
-			(effects
-				(font
-					(size 1.27 1.27)
-				)
-				(justify left)
-			)
-		)
-		(property "Datasheet" ""
-			(at 120.65 88.9 0)
-			(hide yes)
-			(show_name no)
-			(do_not_autoplace no)
-			(effects
-				(font
-					(size 1.27 1.27)
-				)
-			)
-		)
-		(property "Description" "Resettable fuse, polymeric positive temperature coefficient"
-			(at 120.65 88.9 0)
-			(hide yes)
-			(show_name no)
-			(do_not_autoplace no)
-			(effects
-				(font
-					(size 1.27 1.27)
-				)
-			)
-		)
-		(pin "2"
-		)
-		(pin "1"
-		)
-		(instances
-			(project "PWMGenerator_EuniceF"
-				(path "/c15f9de7-7ca4-429e-8134-93b46f4a3e8c"
-					(reference "F1")
-					(unit 1)
-				)
-			)
-		)
-	)
-	(symbol
 		(lib_id "power:PWR_FLAG")
 		(at 74.93 163.83 0)
@@
 					(unit 1)
 				)
+			)
+		)
+	)
+	(symbol
+		(lib_id "Device:Polyfuse")
+		(at 119.38 81.28 90)
+		(unit 1)
+		(body_style 1)
+		(exclude_from_sim no)
+		(in_bom yes)
+		(on_board yes)
+		(in_pos_files yes)
+		(dnp no)
+		(fields_autoplaced yes)
+		(property "Reference" "F1"
+			(at 119.38 74.93 90)
+			(show_name no)
+			(do_not_autoplace no)
+			(effects
+				(font
+					(size 1.27 1.27)
+				)
+			)
+		)
+		(property "Value" "NANOSMDC016F-2"
+			(at 119.38 77.47 90)
+			(show_name no)
+			(do_not_autoplace no)
+			(effects
+				(font
+					(size 1.27 1.27)
+				)
+			)
+		)
+		(property "Footprint" "lib:RESC3115X65N"
+			(at 124.46 80.01 0)
+			(hide yes)
+			(show_name no)
+			(do_not_autoplace no)
+			(effects
+				(font
+					(size 1.27 1.27)
+				)
+				(justify left)
+			)
+		)
+		(property "Datasheet" ""
+			(at 119.38 81.28 0)
+			(hide yes)
+			(show_name no)
+			(do_not_autoplace no)
+			(effects
+				(font
+					(size 1.27 1.27)
+				)
+			)
+		)
+		(property "Description" "Resettable fuse, polymeric positive temperature coefficient"
+			(at 119.38 81.28 0)
+			(hide yes)
+			(show_name no)
+			(do_not_autoplace no)
+			(effects
+				(font
+					(size 1.27 1.27)
+				)
+			)
+		)
+		(pin "1"
+		)
+		(pin "2"
+		)
+		(instances
+			(project "PWMGenerator_EuniceF"
+				(path "/c15f9de7-7ca4-429e-8134-93b46f4a3e8c"
+					(reference "F1")
+					(unit 1)
+				)

Commit message: commit
Parts:
- removed Q1, Q2: 2N3906, Package_TO_SOT_SMD:SOT-23, symbol Transistor_BJT:2N3906
- removed Q5, Q6: 2N3904, Package_TO_SOT_SMD:SOT-23, symbol Device:Q_NPN
- added Q1, Q4: Q_PNP_BCE, Package_TO_SOT_SMD:SOT-23, symbol Transistor_BJT:Q_PNP_BCE
- added Q3, Q7: 2N3904, Package_TO_SOT_SMD:SOT-23, symbol Transistor_BJT:Q_NPN_BCE
- C1, C2: footprint Capacitor_THT:CP_Radial_D10.0mm_P5.00mm_P7.50mm -> Capacitor_THT:C_Disc_D12.5mm_W5.0mm_P10.00mm
Connections:
- net GND: now also Q3.3 (E), Q7.3 (E)
- net PWM: now also Q4.3 (E)
- net VCC 5V: now also Q4.2 (C)
- net at C3.1, U2.4 (-): now also Q1.3 (E), Q7.2 (C)
- net at R4.2: now also Q3.2 (C), Q7.1 (B)
- net at R2.2: now also Q3.1 (B)
- net at R5.2, R6.1: now also Q1.1 (B)
- net at R7.2: now also Q1.2 (C)
- net at R10.2: now also Q4.1 (B)

Commit message: Commit
Connections:
- net GND: now also C1.2, C2.2, U1.2 (GND)
Changed lines of the file:
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@@
 	)
 	(junction
-		(at 161.29 118.11)
-		(diameter 0)
-		(color 0 0 0 0)
-	)
-	(junction
 		(at 215.9 101.6)
 		(diameter 0)
@@
 	)
 	(junction
+		(at 161.29 116.84)
+		(diameter 0)
+		(color 0 0 0 0)
+	)
+	(junction
 		(at 224.79 101.6)
 		(diameter 0)
@@
 	(wire
 		(pts
-			(xy 161.29 118.11) (xy 161.29 121.92)
+			(xy 161.29 116.84) (xy 161.29 121.92)
 		)
 		(stroke
@@
 	(wire
 		(pts
-			(xy 167.64 114.3) (xy 167.64 118.11)
-		)
-		(stroke
-			(width 0)
-			(type default)
-		)
-	)
-	(wire
-		(pts
 			(xy 224.79 139.7) (xy 224.79 142.24)
 		)
@@
 	(wire
 		(pts
-			(xy 167.64 118.11) (xy 161.29 118.11)
+			(xy 205.74 73.66) (xy 240.03 73.66)
 		)
 		(stroke
@@
 	(wire
 		(pts
-			(xy 205.74 73.66) (xy 240.03 73.66)
+			(xy 215.9 133.35) (xy 215.9 140.97)
 		)
 		(stroke
@@
 	(wire
 		(pts
-			(xy 215.9 133.35) (xy 215.9 140.97)
+			(xy 156.21 118.11) (xy 156.21 116.84)
 		)
 		(stroke
@@
 	(wire
 		(pts
-			(xy 161.29 109.22) (xy 161.29 118.11)
+			(xy 161.29 109.22) (xy 161.29 116.84)
 		)
 		(stroke
@@
 	(wire
 		(pts
+			(xy 156.21 116.84) (xy 161.29 116.84)
+		)
+		(stroke
+			(width 0)
+			(type default)
+		)
+	)
+	(wire
+		(pts
 			(xy 157.48 133.35) (xy 165.1 133.35)
 		)
@@
 	)
 	(symbol
+		(lib_id "power:GND")
+		(at 156.21 118.11 0)
+		(unit 1)
+		(body_style 1)
+		(exclude_from_sim no)
+		(in_bom yes)
+		(on_board yes)
+		(in_pos_files yes)
+		(dnp no)
+		(fields_autoplaced yes)
+		(property "Reference" "#PWR04"
+			(at 156.21 124.46 0)
+			(hide yes)
+			(show_name no)
+			(do_not_autoplace no)
+			(effects
+				(font
+					(size 1.27 1.27)
+				)
+			)
+		)
+		(property "Value" "GND"
+			(at 156.21 123.19 0)
+			(show_name no)
+			(do_not_autoplace no)
+			(effects
+				(font
+					(size 1.27 1.27)
+				)
+			)
+		)
+		(property "Footprint" ""
+			(at 156.21 118.11 0)
+			(hide yes)
+			(show_name no)
+			(do_not_autoplace no)
+			(effects
+				(font
+					(size 1.27 1.27)
+				)
+			)
+		)
+		(property "Datasheet" ""
+			(at 156.21 118.11 0)
+			(hide yes)
+			(show_name no)
+			(do_not_autoplace no)
+			(effects
+				(font
+					(size 1.27 1.27)
+				)
+			)
+		)
+		(property "Description" "Power symbol creates a global label with name \"GND\" , ground"
+			(at 156.21 118.11 0)
+			(hide yes)
+			(show_name no)
+			(do_not_autoplace no)
+			(effects
+				(font
+					(size 1.27 1.27)
+				)
+			)
+		)
+		(pin "1"
+		)
+		(instances
+			(project "PWMGenerator_EuniceF"
+				(path "/c15f9de7-7ca4-429e-8134-93b46f4a3e8c"
+					(reference "#PWR04")
+					(unit 1)
+				)
+			)
+		)
+	)
+	(symbol
 		(lib_id "Diode:1N4005")
 		(at 144.78 101.6 180)
@@
 					(unit 1)
 				)
-			)
-		)
-	)
-	(symbol
-		(lib_id "power:PWR_FLAG")
-		(at 167.64 114.3 0)
-		(unit 1)
-		(body_style 1)
-		(exclude_from_sim no)
-		(in_bom yes)
-		(on_board yes)
-		(in_pos_files yes)
-		(dnp no)
-		(fields_autoplaced yes)
-		(property "Reference" "#FLG06"
-			(at 167.64 112.395 0)
-			(hide yes)
-			(show_name no)
-			(do_not_autoplace no)
-			(effects
-				(font
-					(size 1.27 1.27)
-				)
-			)
-		)
-		(property "Value" "PWR_FLAG"
-			(at 167.64 109.22 0)
-			(show_name no)
-			(do_not_autoplace no)
-			(effects
-				(font
-					(size 1.27 1.27)
-				)
-			)
-		)
-		(property "Footprint" ""
-			(at 167.64 114.3 0)
-			(hide yes)
-			(show_name no)
-			(do_not_autoplace no)
-			(effects
-				(font
-					(size 1.27 1.27)
-				)
-			)
-		)
-		(property "Datasheet" ""
-			(at 167.64 114.3 0)
-			(hide yes)
-			(show_name no)
-			(do_not_autoplace no)
-			(effects
-				(font
-					(size 1.27 1.27)
-				)
-			)
-		)
-		(property "Description" "Special symbol for telling ERC where power comes from"
-			(at 167.64 114.3 0)
-			(hide yes)
-			(show_name no)
-			(do_not_autoplace no)
-			(effects
-				(font
-					(size 1.27 1.27)
-				)
-			)
-		)
-		(pin "1"
-		)
-		(instances
-			(project "PWMGenerator_EuniceF"
-				(path "/c15f9de7-7ca4-429e-8134-93b46f4a3e8c"
-					(reference "#FLG06")
-					(unit 1)
-				)
