File: PWMGenerator_EuniceF/PWMGenerator_EuniceF.kicad_pcb (KiCad board)
At the start: 2 copper layers, 0 parts

Commit message: commit
Parts:
- added C1: 220u, Capacitor_THT:C_Disc_D12.5mm_W5.0mm_P10.00mm, F.Cu at (29.5, 156.5)
- added C2: 10u, Capacitor_THT:C_Disc_D12.5mm_W5.0mm_P10.00mm, F.Cu at (29.0, 145.0)
- added C3: 0.1u, Capacitor_SMD:C_0805_2012Metric, F.Cu at (93.0, 75.5)
- added D1: LED_GREEN, LED_THT:LED_D5.0mm-4_RGB, F.Cu at (40.2, 65.5)
- added D2: 1N4005G, Diode_SMD:D_0805_2012Metric, F.Cu at (48.9, 106.0)
- added D3: 1N4005G, Diode_THT:D_DO-41_SOD81_P10.16mm_Horizontal, F.Cu at (40.0, 111.5)
- added D4: 1N4005G, Diode_SMD:D_0805_2012Metric, F.Cu at (47.4, 83.5)
- added D5: 1N4005G, Diode_SMD:D_0805_2012Metric, F.Cu at (41.4, 120.5)
- added D6: 1N4005G, Diode_SMD:D_0805_2012Metric, F.Cu at (40.1, 104.5)
- added F1: NANOSMDC016F-2, lib:RESC3115X65N, F.Cu at (38.0, 81.0)
- added J1: Conn_01x03_Pin, Connector_PinHeader_2.54mm:PinHeader_1x03_P2.54mm_Horizontal, F.Cu at (133.5, 85.1)
- added J2: Barrel_Jack, Connector_BarrelJack:BarrelJack_CUI_PJ-063AH_Horizontal, F.Cu at (24.5, 93.5)
- added Q1: Q_PNP_BCE, Package_TO_SOT_SMD:SOT-23, F.Cu at (78.4, 109.0)
- added Q3: 2N3904, Package_TO_SOT_SMD:SOT-23, F.Cu at (72.4, 75.0)
- added Q4: Q_PNP_BCE, Package_TO_SOT_SMD:SOT-23, F.Cu at (150.4, 83.9)
- added Q7: 2N3904, Package_TO_SOT_SMD:SOT-23, F.Cu at (74.0, 86.4)
- added R1: 2.2k, Resistor_SMD:R_0805_2012Metric, F.Cu at (135.1, 57.5)
- added R10: 8.2k, Resistor_SMD:R_0805_2012Metric, F.Cu at (150.4, 94.0)
- added R11: 180, Resistor_SMD:R_0805_2012Metric, F.Cu at (122.4, 68.0)
- added R2: 1M, Resistor_SMD:R_0805_2012Metric, F.Cu at (71.5, 66.9)
- added R3: 330, Resistor_SMD:R_0805_2012Metric, F.Cu at (65.6, 64.5)
- added R4: 10k, Resistor_SMD:R_0805_2012Metric, F.Cu at (103.4, 99.5)
- added R5: 220k, Resistor_SMD:R_0805_2012Metric, F.Cu at (66.9, 116.0)
- added R6: 390, Resistor_SMD:R_0805_2012Metric, F.Cu at (57.6, 113.0)
- added R7: 22k, Resistor_SMD:R_0805_2012Metric, F.Cu at (67.9, 101.5)
- added R8: 2.2k, Resistor_SMD:R_0805_2012Metric, F.Cu at (59.9, 130.5)
- added RV1: 5k, Potentiometer_THT:Potentiometer_ACP_CA14-H2,5_Horizontal, F.Cu at (130.5, 119.0)
- added SW1: SW_SPST, Button_Switch_SMD:SW_DIP_SPSTx01_Slide_6.7x4.1mm_W6.73mm_P2.54mm_LowProfile_JPin, F.Cu at (24.5, 67.9)
- added U1: LM7805_TO220, Package_TO_SOT_THT:TO-220-3_Horizontal_TabDown, F.Cu at (22.5, 131.7)
- added U2: LM339, Package_SO:SOIC-14_3.9x8.7mm_P1.27mm, F.Cu at (104.0, 119.0)

Commit message: Commit
Parts:
- moved R1 49.3 mm to (87.4, 70.0)
- moved C1 44.4 mm to (52.5, 118.5)
- moved C2 41.3 mm to (44.0, 106.5)
- moved D5 40.0 mm to (40.6, 80.5)
- moved R10 37.6 mm to (112.9, 91.5)
- moved J1 34.2 mm to (99.5, 88.5)
- moved Q4 29.0 mm to (121.5, 85.4)
- moved RV1 28.6 mm to (103.0, 111.0)
- moved R11 27.9 mm to (95.4, 75.0)
- moved Q1 26.9 mm to (58.1, 91.5)
- moved U2 24.1 mm to (83.5, 106.3)
- moved R4 23.4 mm to (81.4, 91.5)
- moved D2 23.2 mm to (35.0, 87.4), turned to 90 degrees
- moved R8 22.2 mm to (54.5, 109.0)
- moved R5 16.7 mm to (62.0, 100.0), turned to 180 degrees
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Connections:
- C1 pad 2: Net-(U1-GND) -> GND
- C2 pad 2: Net-(U1-GND) -> GND
- U1 pad 2: Net-(U1-GND) -> GND
Routing:
- net VCC 5V: track 0.00 -> 269.4 mm
- net GND: track 0.00 -> 211.5 mm
- net Net-(D3-K): track 0.00 -> 81.1 mm
- net Net-(D5-K): track 0.00 -> 77.1 mm
- net Net-(U2A-+): track 0.00 -> 74.6 mm
- net Net-(D4-K): track 0.00 -> 66.0 mm
- net Net-(Q1-E): track 0.00 -> 48.8 mm
- net PWM: track 0.00 -> 42.0 mm
- net Net-(R10-Pad1): track 0.00 -> 36.1 mm
- net Net-(D2-K): track 0.00 -> 23.3 mm
- net Net-(Q3-B): track 0.00 -> 17.7 mm
- net Net-(D1-A): track 0.00 -> 16.7 mm
- net Net-(Q3-C): track 0.00 -> 9.72 mm
- added copper zone on B.Cu, net GND
- added copper zone on F.Cu, net VCC 5V

Commit message: PCB Part C COMMIT
Parts:
- moved R4 27.6 mm to (55.5, 82.0)
- moved Q1 11.4 mm to (68.9, 88.0)
- moved R3 9.36 mm to (49.5, 65.0)
- moved R1 7.28 mm to (80.4, 68.0)
- moved U2 5.95 mm to (78.0, 108.5)
- moved R2 5.78 mm to (72.0, 74.1)
- moved D2 4.87 mm to (33.0, 83.0), turned to 0 degrees
- moved R5 1.00 mm to (62.0, 101.0)
- moved RV1 0.50 mm to (102.5, 111.0)
- turned D4 to -90 degrees
- turned D6 to 180 degrees
- turned R6 to 180 degrees
- turned R8 to -90 degrees
Routing:
- net VCC 5V: track 269.4 -> 0.00 mm
- net GND: track 211.5 -> 1.28 mm
- net Net-(D3-K): track 81.1 -> 1.10 mm
- net Net-(D5-K): track 77.1 -> 0.00 mm
- net Net-(U2A-+): track 74.6 -> 0.00 mm
- net Net-(D4-K): track 66.0 -> 0.00 mm
- net Net-(Q1-E): track 48.8 -> 0.00 mm
- net PWM: track 42.0 -> 0.00 mm
- net Net-(R10-Pad1): track 36.1 -> 0.00 mm
- net Net-(D2-K): track 23.3 -> 0.01 mm
- net Net-(Q3-B): track 17.7 -> 0.00 mm
- net Net-(Q3-C): track 9.72 -> 0.00 mm
- net Net-(D1-A): track 16.7 -> 10.7 mm
- net Net-(Q1-C): track 0.00 -> 0.50 mm
- net Net-(Q1-B): track 0.00 -> 0.50 mm

Commit message: PCB PARTC WORKING
Parts:
- moved R8 64.5 mm to (119.0, 109.5)
- moved D3 25.2 mm to (40.5, 72.4), turned to -90 degrees
- moved R6 23.1 mm to (69.5, 79.0)
- moved R7 18.6 mm to (82.5, 94.0)
- moved R2 18.2 mm to (55.5, 66.5), turned to -90 degrees
- moved D5 17.7 mm to (35.5, 97.5)
- moved C3 17.2 mm to (66.5, 73.5)
- moved R5 14.7 mm to (74.6, 93.5)
- moved D4 8.58 mm to (32.5, 90.0), turned to 90 degrees
- moved D2 2.50 mm to (34.5, 81.0), turned to 90 degrees
- moved J1 2.00 mm to (97.5, 88.6)
- moved R3 0.71 mm to (49.0, 64.5)
- turned F1 to 90 degrees
- turned Q4 to 90 degrees
- turned R11 to 180 degrees
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Routing:
- net GND: track 1.28 -> 87.9 mm
- net Net-(D3-K): track 1.10 -> 82.5 mm
- net Net-(D4-K): track 0.00 -> 67.2 mm
- net Net-(D5-K): track 0.00 -> 56.2 mm
- net Net-(U2A-+): track 0.00 -> 44.2 mm
- net Net-(Q1-E): track 0.00 -> 44.2 mm
- net Net-(R10-Pad1): track 0.00 -> 42.5 mm
- net PWM: track 0.00 -> 40.3 mm
- net VCC 5V: track 0.00 -> 26.3 mm
- net Net-(D2-K): track 0.01 -> 17.8 mm
- net Net-(Q1-B): track 0.50 -> 17.2 mm
- net Net-(Q3-C): track 0.00 -> 14.3 mm
- net Net-(Q1-C): track 0.50 -> 14.6 mm
- net Net-(SW1-B): track 0.00 -> 10.0 mm
- net Net-(Q4-B): track 0.00 -> 8.80 mm
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Other:
- board outline added: 111.5 x 64.5 mm

Commit message: Partc Final working
Parts:
- moved C1 18.6 mm to (34.0, 116.5), turned to 0 degrees
- moved C2 10.3 mm to (53.0, 101.5)
Routing:
- net VCC 5V: track 26.3 -> 147.3 mm
- net Net-(D5-K): track 56.2 -> 42.6 mm
Other:
- board size 111.5 x 64.5 mm -> 111 x 65.4 mm
Changed lines of the file:
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@@
 	(footprint "Capacitor_THT:C_Disc_D12.5mm_W5.0mm_P10.00mm"
 		(layer "F.Cu")
-		(at 44 106.5 180)
+		(at 53 101.5 180)
 		(descr "C, Disc series, Radial, pin pitch=10.00mm, diameter*width=12.5*5.0mm^2, Capacitor, http://www.vishay.com/docs/28535/vy2series.pdf")
 		(tags "C Disc series Radial pin pitch 10.00mm diameter 12.5mm width 5.0mm Capacitor")
@@
 	(footprint "Capacitor_THT:C_Disc_D12.5mm_W5.0mm_P10.00mm"
 		(layer "F.Cu")
-		(at 52.5 118.5 180)
+		(at 34 116.5)
 		(descr "C, Disc series, Radial, pin pitch=10.00mm, diameter*width=12.5*5.0mm^2, Capacitor, http://www.vishay.com/docs/28535/vy2series.pdf")
 		(tags "C Disc series Radial pin pitch 10.00mm diameter 12.5mm width 5.0mm Capacitor")
@@
 		(duplicate_pad_numbers_are_jumpers no)
 		(fp_line
-			(start 11.37 2.62)
-			(end -1.37 2.62)
+			(start -1.37 -2.62)
+			(end 11.37 -2.62)
 			(stroke
 				(width 0.12)
@@
 		)
 		(fp_line
-			(start 11.37 -2.62)
-			(end 11.37 2.62)
+			(start -1.37 2.62)
+			(end -1.37 -2.62)
 			(stroke
 				(width 0.12)
@@
 		)
 		(fp_line
-			(start -1.37 2.62)
-			(end -1.37 -2.62)
+			(start 11.37 -2.62)
+			(end 11.37 2.62)
 			(stroke
 				(width 0.12)
@@
 		)
 		(fp_line
-			(start -1.37 -2.62)
-			(end 11.37 -2.62)
+			(start 11.37 2.62)
+			(end -1.37 2.62)
 			(stroke
 				(width 0.12)
@@
 		)
 		(pad "1" thru_hole circle
-			(at 0 0 180)
+			(at 0 0)
 			(size 2 2)
 			(drill 1)
@@
 		)
 		(pad "2" thru_hole circle
-			(at 10 0 180)
+			(at 10 0)
 			(size 2 2)
 			(drill 1)
@@
 	(gr_rect
 		(start 15 60)
-		(end 126.5 124.5)
+		(end 125.972102 125.397888)
 		(stroke
 			(width 0.05)
@@
 	)
 	(segment
+		(start 76.775 108.880552)
+		(end 76.775 106.859448)
+		(width 0.2)
+		(layer "F.Cu")
+		(net "VCC 5V")
+	)
+	(segment
+		(start 76.515552 109.14)
+		(end 76.775 108.880552)
+		(width 0.2)
+		(layer "F.Cu")
+		(net "VCC 5V")
+	)
+	(segment
+		(start 26.18 119.8)
+		(end 26.04 119.66)
+		(width 0.2)
+		(layer "F.Cu")
+		(net "VCC 5V")
+	)
+	(segment
+		(start 74.544381 106.659933)
+		(end 74.225 106.340552)
+		(width 0.2)
+		(layer "F.Cu")
+		(net "VCC 5V")
+	)
+	(segment
+		(start 26.04 119.66)
+		(end 47.84 119.66)
+		(width 0.2)
+		(layer "F.Cu")
+		(net "VCC 5V")
+	)
+	(segment
 		(start 91.3725 86.04)
 		(end 83.4125 94)
@@
 	)
 	(segment
+		(start 54.5 103)
+		(end 53 101.5)
+		(width 0.2)
+		(layer "F.Cu")
+		(net "VCC 5V")
+	)
+	(segment
+		(start 54.5875 89.243052)
+		(end 74.484448 109.14)
+		(width 0.2)
+		(layer "F.Cu")
+		(net "VCC 5V")
+	)
+	(segment
+		(start 74.225 106.340552)
+		(end 74.225 103.1875)
+		(width 0.2)
+		(layer "F.Cu")
+		(net "VCC 5V")
+	)
+	(segment
+		(start 53 101.5)
+		(end 53 101)
+		(width 0.2)
+		(layer "F.Cu")
+		(net "VCC 5V")
+	)
+	(segment
 		(start 82.4125 95)
 		(end 83.4125 94)
@@
 	)
 	(segment
+		(start 54.5 113)
+		(end 54.5 103)
+		(width 0.2)
+		(layer "F.Cu")
+		(net "VCC 5V")
+	)
+	(segment
+		(start 76.775 106.859448)
+		(end 76.575485 106.659933)
+		(width 0.2)
+		(layer "F.Cu")
+		(net "VCC 5V")
+	)
+	(segment
+		(start 54.5875 99.4125)
+		(end 54.5875 82)
+		(width 0.2)
+		(layer "F.Cu")
+		(net "VCC 5V")
+	)
+	(segment
+		(start 47.84 119.66)
+		(end 54.5 113)
+		(width 0.2)
+		(layer "F.Cu")
+		(net "VCC 5V")
+	)
+	(segment
+		(start 76.575485 106.659933)
+		(end 74.544381 106.659933)
+		(width 0.2)
+		(layer "F.Cu")
+		(net "VCC 5V")
+	)
+	(segment
 		(start 97.5 86.04)
 		(end 91.3725 86.04)
@@
 	)
 	(segment
+		(start 74.484448 109.14)
+		(end 76.515552 109.14)
+		(width 0.2)
+		(layer "F.Cu")
+		(net "VCC 5V")
+	)
+	(segment
 		(start 77 95)
 		(end 82.4125 95)
@@
 	)
 	(segment
+		(start 74.225 103.1875)
+		(end 82.4125 95)
+		(width 0.2)
+		(layer "F.Cu")
+		(net "VCC 5V")
+	)
+	(segment
+		(start 54.5875 82)
+		(end 54.5875 89.243052)
+		(width 0.2)
+		(layer "F.Cu")
+		(net "VCC 5V")
+	)
+	(segment
+		(start 53 101)
+		(end 54.5875 99.4125)
+		(width 0.2)
+		(layer "F.Cu")
+		(net "VCC 5V")
+	)
+	(segment
 		(start 68.8375 80.575)
 		(end 68.8375 87.390552)
@@
 	)
 	(segment
-		(start 34.5625 97.5)
-		(end 34.5625 100.5625)
+		(start 24.12 116.5)
+		(end 20.96 119.66)
 		(width 0.2)
 		(layer "F.Cu")
@@
 	)
 	(segment
-		(start 34.5625 100.5625)
-		(end 52.5 118.5)
+		(start 34.5 116.5)
+		(end 24.12 116.5)
 		(width 0.2)
 		(layer "F.Cu")
@@
 		(polygon
 			(pts
-				(xy 15 60) (xy 126 60) (xy 126 125) (xy 15 125)
+				(xy 15 60) (xy 126 60) (xy 126 125.5) (xy 15 125.5)
 			)
 		)
@@
 		(min_thickness 0.25)
 		(fill yes
+			(mode hatch)
 			(thermal_gap 0.5)
 			(thermal_bridge_width 0.5)
 			(island_removal_mode 0)
+			(hatch_thickness 1)
+			(hatch_gap 1.5)
+			(hatch_orientation 0)
+			(hatch_border_algorithm hatch_thickness)
+			(hatch_min_hole_area 0.15)
 		)
 		(polygon
 			(pts
-				(xy 15 60) (xy 126 60) (xy 126 125) (xy 15 125)
+				(xy 15 60) (xy 126 60) (xy 126 125.5) (xy 15 125.5)
 			)
 		)
